File: hardware/jack_plate/kicad_7/ribbon_controller_jack_plate.kicad_pcb (KiCad board)
At the start: 2 copper layers, 110.6 x 21.7 mm, 0 parts

Commit message: Design jack plate
Parts:
- added H1: MountingHole_Pad, MountingHole:MountingHole_3.2mm_M3_Pad_Via, F.Cu at (60.3, 85.7)
- added H2: MountingHole_Pad, MountingHole:MountingHole_3.2mm_M3_Pad_Via, F.Cu at (60.3, 111.8)
- added H3: MountingHole_Pad, MountingHole:MountingHole_3.2mm_M3_Pad_Via, F.Cu at (240.0, 85.7)
- added H4: MountingHole_Pad, MountingHole:MountingHole_3.2mm_M3_Pad_Via, F.Cu at (240.0, 111.8)
Routing:
- added copper zone on B.Cu, net GND
- added copper zone on F.Cu, net GND
Other:
- board size 110.6 x 21.7 mm -> 188.6 x 34.9 mm
- board text added: "CV-MIDI RIBBON CONTROLLER"
- board text added: "JLCJLCJLCJLC"
- board text added: "MIDI OUT"
- board text added: "github.com/JordanAceto/rust_ribbon_controller"
- board text removed: "MIDI IN"
- board text removed: "TODO: Front panel barely started These are roughly the right number of holes, but they are not necessarily the right size or position."
